File: Southpaw/Southpaw.sch (KiCad schematic (older format))
At the start: 162 parts

Commit message: Duplex
Parts:
- removed D? (x50): BAV70, Package_TO_SOT_SMD:SOT-23, symbol Diode:BAV70
- removed SW? (x100): SW_Push, symbol Switch:SW_Push
- added D1, D10, D11, D12, D13, D14, D15, D16, D17, D18, D19, D2, D20, D21, D22, D23, D24, D25, D26, D27, D28, D29, D3, D30, D31, D32, D33, D34, D35, D36, D37, D38, D39, D4, D40, D41, D42, D43, D44, D45, D46, D47, D48, D5, D6, D7, D8, D9: BAV70, Package_TO_SOT_SMD:SOT-23, symbol Diode:BAV70
- added SW1: NMLK, symbol Switch:SW_Push
- added SW10, SW5, SW65: 0, symbol Switch:SW_Push
- added SW11: Mult, symbol Switch:SW_Push
- added SW12, SW61: 9, symbol Switch:SW_Push
- added SW13, SW48: 6, symbol Switch:SW_Push
- added SW14, SW36: 3, symbol Switch:SW_Push
- added SW15, SW68: Dot, symbol Switch:SW_Push
- added SW16, SW70: Sub, symbol Switch:SW_Push
- added SW17, SW18, SW75: Add, symbol Switch:SW_Push
- added SW19, SW20, SW77: Enter, symbol Switch:SW_Push
- added SW2, SW53: 7, symbol Switch:SW_Push
- added SW21: Esc, symbol Switch:SW_Push
- added SW22: Tab, symbol Switch:SW_Push
- added SW23: Caps, symbol Switch:SW_Push
- added SW24, SW29, SW78: Shift, symbol Switch:SW_Push
- added SW25, SW79: Ctrl, symbol Switch:SW_Push
- added SW26, SW4: 1, symbol Switch:SW_Push
- added SW27: Q, symbol Switch:SW_Push
- added SW28: A, symbol Switch:SW_Push
- added SW3, SW40: 4, symbol Switch:SW_Push
- added SW30, SW74: Win, symbol Switch:SW_Push
- added SW31, SW9: 2, symbol Switch:SW_Push
- added SW32: W, symbol Switch:SW_Push
- added SW33: S, symbol Switch:SW_Push
- added SW34: Z, symbol Switch:SW_Push
- added SW35, SW69: Alt, symbol Switch:SW_Push
- added SW37: E, symbol Switch:SW_Push
- added SW38: D, symbol Switch:SW_Push
- added SW39: X, symbol Switch:SW_Push
- added SW41: R, symbol Switch:SW_Push
- added SW42: F, symbol Switch:SW_Push
- added SW43: C, symbol Switch:SW_Push
- added SW44, SW8: 5, symbol Switch:SW_Push
- added SW45: T, symbol Switch:SW_Push
- added SW46: G, symbol Switch:SW_Push
- added SW47: V, symbol Switch:SW_Push
- added SW49: Y, symbol Switch:SW_Push
- added SW50: H, symbol Switch:SW_Push
- added SW51: B, symbol Switch:SW_Push
- added SW52: Space, symbol Switch:SW_Push
- added SW54: U, symbol Switch:SW_Push
- added SW55: J, symbol Switch:SW_Push
- added SW56: N, symbol Switch:SW_Push
- added SW57, SW7: 8, symbol Switch:SW_Push
- added SW58: I, symbol Switch:SW_Push
- added SW59: K, symbol Switch:SW_Push
- added SW6: Div, symbol Switch:SW_Push
- added SW60: M, symbol Switch:SW_Push
- added SW62: O, symbol Switch:SW_Push
- added SW63: L, symbol Switch:SW_Push
- added SW64: Comm, symbol Switch:SW_Push
- added SW66: P, symbol Switch:SW_Push
- added SW67: SCLN, symbol Switch:SW_Push
- added SW71: LBrac, symbol Switch:SW_Push
- added SW72: Quote, symbol Switch:SW_Push
- added SW73: Slash, symbol Switch:SW_Push
- added SW76: RBrac, symbol Switch:SW_Push
- added SW80, SW81: Pipe, symbol Switch:SW_Push
- added SW82: Left, symbol Switch:SW_Push
- added SW83: Backspace, symbol Switch:SW_Push
- added SW84: Up, symbol Switch:SW_Push
- added SW85: Down, symbol Switch:SW_Push
- added SW86: Mute, symbol Switch:SW_Push
- added SW87: Del, symbol Switch:SW_Push
- added SW88: End, symbol Switch:SW_Push
- added SW89: Home, symbol Switch:SW_Push
- added SW90: Right, symbol Switch:SW_Push
- gave numbers to parts that had none: 12
Connections:
- net col0: now also D1.3 (K), D2.3 (K), D3.3 (K), D4.3 (K), D5.3 (K)
- net col1: now also D10.3 (K), D6.3 (K), D7.3 (K), D8.3 (K), D9.3 (K)
- net col2: now also D11.3 (K), D12.3 (K), D13.3 (K), D14.3 (K), D15.3 (K)
- net col3: now also D16.3 (K), D17.3 (K), D18.3 (K), D19.3 (K), D20.3 (K)
- net col4: now also D21.3 (K), D22.3 (K), D23.3 (K), D24.3 (K)
- net col5: now also D25.3 (K), D26.3 (K), D27.3 (K), D28.3 (K), D29.3 (K)
- net col6: now also D30.3 (K), D31.3 (K), D32.3 (K), D33.3 (K)
- net col7: now also D34.3 (K), D35.3 (K), D36.3 (K), D37.3 (K), D38.3 (K)
- net col8: now also D39.3 (K), D40.3 (K), D41.3 (K), D42.3 (K), D43.3 (K)
- net col9: now also D44.3 (K), D45.3 (K), D46.3 (K), D47.3 (K), D48.3 (K)
- net row0: now also SW1.1, SW11.1, SW21.1, SW31.1, SW40.1, SW48.1, SW57.1, SW65.1, SW75.1, SW83.1
- net row1: now also SW16.1, SW26.1, SW36.1, SW44.1, SW53.1, SW6.1, SW61.1, SW70.1, SW80.1, SW86.1
- net row2: now also SW12.1, SW2.1, SW22.1, SW32.1, SW41.1, SW49.1, SW58.1, SW66.1, SW76.1
- net row3: now also SW17.1, SW27.1, SW37.1, SW45.1, SW54.1, SW62.1, SW7.1, SW71.1, SW81.1, SW87.1
- net row4: now also SW13.1, SW23.1, SW3.1, SW33.1, SW42.1, SW50.1, SW59.1, SW67.1, SW77.1
- net row5: now also SW18.1, SW28.1, SW38.1, SW46.1, SW55.1, SW63.1, SW72.1, SW8.1, SW88.1
- net row6: now also SW14.1, SW24.1, SW34.1, SW4.1, SW43.1, SW51.1, SW60.1, SW68.1, SW78.1, SW84.1
- net row7: now also SW19.1, SW29.1, SW39.1, SW47.1, SW56.1, SW64.1, SW73.1, SW89.1, SW9.1
- net row8: now also SW15.1, SW25.1, SW35.1, SW5.1, SW52.1, SW69.1, SW79.1, SW85.1
- net row9: now also SW10.1, SW20.1, SW30.1, SW74.1, SW82.1, SW90.1
- new net: D1.1 (A), SW1.2
- new net: D1.2 (A), SW6.2
- new net: D2.1 (A), SW2.2
- new net: D2.2 (A), SW7.2
- new net: D3.1 (A), SW3.2
- new net: D3.2 (A), SW8.2
- new net: D4.1 (A), SW4.2
- new net: D4.2 (A), SW9.2
- new net: D5.1 (A), SW5.2
- new net: D5.2 (A), SW10.2
- new net: D6.1 (A), SW11.2
- new net: D6.2 (A), SW16.2
- new net: D7.1 (A), SW12.2
- new net: D7.2 (A), SW17.2
- new net: D8.1 (A), SW13.2
- new net: D8.2 (A), SW18.2
- new net: D9.1 (A), SW14.2
- new net: D9.2 (A), SW19.2
- new net: D10.1 (A), SW15.2
- new net: D10.2 (A), SW20.2
- new net: D11.1 (A), SW21.2
- new net: D11.2 (A), SW26.2
- new net: D12.1 (A), SW22.2
- new net: D12.2 (A), SW27.2
- new net: D13.1 (A), SW23.2
- new net: D13.2 (A), SW28.2
- new net: D14.1 (A), SW24.2
- new net: D14.2 (A), SW29.2
- new net: D15.1 (A), SW25.2
- new net: D15.2 (A), SW30.2
- new net: D16.1 (A), SW31.2
- new net: D16.2 (A), SW36.2
- new net: D17.1 (A), SW32.2
- new net: D17.2 (A), SW37.2
- new net: D18.1 (A), SW33.2
- new net: D18.2 (A), SW38.2
- new net: D19.1 (A), SW34.2
- new net: D19.2 (A), SW39.2
- new net: D20.1 (A), SW35.2
- new net: D21.1 (A), SW40.2
- new net: D21.2 (A), SW44.2
- new net: D22.1 (A), SW41.2
- new net: D22.2 (A), SW45.2
- new net: D23.1 (A), SW42.2
- new net: D23.2 (A), SW46.2
- new net: D24.1 (A), SW43.2
- new net: D24.2 (A), SW47.2
- new net: D25.1 (A), SW48.2
- new net: D25.2 (A), SW53.2
- new net: D26.1 (A), SW49.2
- new net: D26.2 (A), SW54.2
- new net: D27.1 (A), SW50.2
- new net: D27.2 (A), SW55.2
- new net: D28.1 (A), SW51.2
- new net: D28.2 (A), SW56.2
- new net: D29.1 (A), SW52.2
- new net: D30.1 (A), SW57.2
- new net: D30.2 (A), SW61.2
- new net: D31.1 (A), SW58.2
- new net: D31.2 (A), SW62.2
- new net: D32.1 (A), SW59.2
- new net: D32.2 (A), SW63.2
- new net: D33.1 (A), SW60.2
- new net: D33.2 (A), SW64.2
- new net: D34.1 (A), SW65.2
- new net: D34.2 (A), SW70.2
- new net: D35.1 (A), SW66.2
- new net: D35.2 (A), SW71.2
- new net: D36.1 (A), SW67.2
- new net: D36.2 (A), SW72.2
- new net: D37.1 (A), SW68.2
- new net: D37.2 (A), SW73.2
- new net: D38.1 (A), SW69.2
- new net: D38.2 (A), SW74.2
- new net: D39.1 (A), SW75.2
- new net: D39.2 (A), SW80.2
- new net: D40.1 (A), SW76.2
- new net: D40.2 (A), SW81.2
- new net: D41.1 (A), SW77.2
- new net: D42.1 (A), SW78.2
- new net: D43.1 (A), SW79.2
- new net: D43.2 (A), SW82.2
- new net: D44.1 (A), SW83.2
- new net: D44.2 (A), SW86.2
- new net: D45.2 (A), SW87.2
- new net: D46.2 (A), SW88.2
- new net: D47.1 (A), SW84.2
- new net: D47.2 (A), SW89.2
- new net: D48.1 (A), SW85.2
- new net: D48.2 (A), SW90.2
Other:
- moved on the sheet: C1, C2, C3, C4, C5, R1, R2, R3, R4, RST1, U1, Y1

Commit message: Layout
Parts:
- removed SW1: NMLK, symbol Switch:SW_Push
- removed SW10, SW5, SW65: 0, symbol Switch:SW_Push
- removed SW11: Mult, symbol Switch:SW_Push
- removed SW12, SW61: 9, symbol Switch:SW_Push
- removed SW13, SW48: 6, symbol Switch:SW_Push
- removed SW14, SW36: 3, symbol Switch:SW_Push
- removed SW15, SW68: Dot, symbol Switch:SW_Push
- removed SW16, SW70: Sub, symbol Switch:SW_Push
- removed SW17, SW18, SW75: Add, symbol Switch:SW_Push
- removed SW19, SW20, SW77: Enter, symbol Switch:SW_Push
- removed SW2, SW53: 7, symbol Switch:SW_Push
- removed SW21: Esc, symbol Switch:SW_Push
- removed SW22: Tab, symbol Switch:SW_Push
- removed SW23: Caps, symbol Switch:SW_Push
- removed SW24, SW29, SW78: Shift, symbol Switch:SW_Push
- removed SW25, SW79: Ctrl, symbol Switch:SW_Push
- removed SW26, SW4: 1, symbol Switch:SW_Push
- removed SW27: Q, symbol Switch:SW_Push
- removed SW28: A, symbol Switch:SW_Push
- removed SW3, SW40: 4, symbol Switch:SW_Push
- removed SW30, SW74: Win, symbol Switch:SW_Push
- removed SW31, SW9: 2, symbol Switch:SW_Push
- removed SW32: W, symbol Switch:SW_Push
- removed SW33: S, symbol Switch:SW_Push
- removed SW34: Z, symbol Switch:SW_Push
- removed SW35, SW69: Alt, symbol Switch:SW_Push
- removed SW37: E, symbol Switch:SW_Push
- removed SW38: D, symbol Switch:SW_Push
- removed SW39: X, symbol Switch:SW_Push
- removed SW41: R, symbol Switch:SW_Push
- removed SW42: F, symbol Switch:SW_Push
- removed SW43: C, symbol Switch:SW_Push
- removed SW44, SW8: 5, symbol Switch:SW_Push
- removed SW45: T, symbol Switch:SW_Push
- removed SW46: G, symbol Switch:SW_Push
- removed SW47: V, symbol Switch:SW_Push
- removed SW49: Y, symbol Switch:SW_Push
- removed SW50: H, symbol Switch:SW_Push
- removed SW51: B, symbol Switch:SW_Push
- removed SW52: Space, symbol Switch:SW_Push
- removed SW54: U, symbol Switch:SW_Push
- removed SW55: J, symbol Switch:SW_Push
- removed SW56: N, symbol Switch:SW_Push
- removed SW57, SW7: 8, symbol Switch:SW_Push
- removed SW58: I, symbol Switch:SW_Push
- removed SW59: K, symbol Switch:SW_Push
- removed SW6: Div, symbol Switch:SW_Push
- removed SW60: M, symbol Switch:SW_Push
- removed SW62: O, symbol Switch:SW_Push
- removed SW63: L, symbol Switch:SW_Push
- removed SW64: Comm, symbol Switch:SW_Push
- removed SW66: P, symbol Switch:SW_Push
- removed SW67: SCLN, symbol Switch:SW_Push
- removed SW71: LBrac, symbol Switch:SW_Push
- removed SW72: Quote, symbol Switch:SW_Push
- removed SW73: Slash, symbol Switch:SW_Push
- removed SW76: RBrac, symbol Switch:SW_Push
- removed SW80, SW81: Pipe, symbol Switch:SW_Push
- removed SW82: Left, symbol Switch:SW_Push
- removed SW83: Backspace, symbol Switch:SW_Push
- removed SW84: Up, symbol Switch:SW_Push
- removed SW85: Down, symbol Switch:SW_Push
- removed SW86: Mute, symbol Switch:SW_Push
- removed SW87: Del, symbol Switch:SW_Push
- removed SW88: End, symbol Switch:SW_Push
- removed SW89: Home, symbol Switch:SW_Push
- removed SW90: Right, symbol Switch:SW_Push
- added C6: 4.7nF, Custom_Footprints:C_0603_Annotated, symbol Device:C_Small
- added F1: 500mA, Custom_Footprints:Fuse_1206_Annotated, symbol Device:Polyfuse_Small
- added J1: USB C, Custom_Footprints:Mid_Mount-USB_C_HandSoldering, symbol Connector:USB_C_Receptacle_USB2.0
- added K1: Num, MX_Only:MXOnly-1U-NoLED, symbol Switch:SW_Push
- added K10, K43: 5, MX_Only:MXOnly-1U-NoLED, symbol Switch:SW_Push
- added K11, K44: 6, MX_Only:MXOnly-1U-NoLED, symbol Switch:SW_Push
- added K12, K22: 7, MX_Only:MXOnly-1U-NoLED, symbol Switch:SW_Push
- added K13, K23: 8, MX_Only:MXOnly-1U-NoLED, symbol Switch:SW_Push
- added K14, K24: 9, MX_Only:MXOnly-1U-NoLED, symbol Switch:SW_Push
- added K15: 0, MX_Only:MXOnly-1U-NoLED, symbol Switch:SW_Push
- added K16, K4: Sub, MX_Only:MXOnly-1U-NoLED, symbol Switch:SW_Push
- added K17: Plus, MX_Only:MXOnly-1U-NoLED, symbol Switch:SW_Push
- added K18: Backspace, MX_Only:MXOnly-2U-NoLED, symbol Switch:SW_Push
- added K19, K40: Del, MX_Only:MXOnly-1U-NoLED, symbol Switch:SW_Push
- added K2, K75: Slash, MX_Only:MXOnly-1U-NoLED, symbol Switch:SW_Push
- added K20: Mute, MX_Only:MXOnly-1U-NoLED, symbol Switch:SW_Push
- added K21: Backspace, MX_Only:MXOnly-1U-NoLED, symbol Switch:SW_Push
- added K25: Plus, MX_Only:MXOnly-2U-NoLED, symbol Switch:SW_Push
- added K26: Tab, MX_Only:MXOnly-1.5U-NoLED, symbol Switch:SW_Push
- added K27: Q, MX_Only:MXOnly-1U-NoLED, symbol Switch:SW_Push
- added K28: W, MX_Only:MXOnly-1U-NoLED, symbol Switch:SW_Push
- added K29: E, MX_Only:MXOnly-1U-NoLED, symbol Switch:SW_Push
- added K3: Mult, MX_Only:MXOnly-1U-NoLED, symbol Switch:SW_Push
- added K30: R, MX_Only:MXOnly-1U-NoLED, symbol Switch:SW_Push
- added K31: T, MX_Only:MXOnly-1U-NoLED, symbol Switch:SW_Push
- added K32: Y, MX_Only:MXOnly-1U-NoLED, symbol Switch:SW_Push
- added K33: U, MX_Only:MXOnly-1U-NoLED, symbol Switch:SW_Push
- added K34: I, MX_Only:MXOnly-1U-NoLED, symbol Switch:SW_Push
- added K35: O, MX_Only:MXOnly-1U-NoLED, symbol Switch:SW_Push
- added K36: P, MX_Only:MXOnly-1U-NoLED, symbol Switch:SW_Push
- added K37: LBrac, MX_Only:MXOnly-1U-NoLED, symbol Switch:SW_Push
- added K38: Rbrac, MX_Only:MXOnly-1U-NoLED, symbol Switch:SW_Push
- added K39: Pipe, MX_Only:MXOnly-1.5U-NoLED, symbol Switch:SW_Push
- added K41: SCaps, MX_Only:MXOnly-1.25U-NoLED, symbol Switch:SW_Push
- added K42, K9: 4, MX_Only:MXOnly-1U-NoLED, symbol Switch:SW_Push
- added K45: Caps, MX_Only:MXOnly-1.75U-NoLED, symbol Switch:SW_Push
- added K46: A, MX_Only:MXOnly-1U-NoLED, symbol Switch:SW_Push
- added K47: S, MX_Only:MXOnly-1U-NoLED, symbol Switch:SW_Push
- added K48: D, MX_Only:MXOnly-1U-NoLED, symbol Switch:SW_Push
- added K49: F, MX_Only:MXOnly-1U-NoLED, symbol Switch:SW_Push
- added K5: Esc, MX_Only:MXOnly-1U-NoLED, symbol Switch:SW_Push
- added K50: G, MX_Only:MXOnly-1U-NoLED, symbol Switch:SW_Push
- added K51: H, MX_Only:MXOnly-1U-NoLED, symbol Switch:SW_Push
- added K52: J, MX_Only:MXOnly-1U-NoLED, symbol Switch:SW_Push
- added K53: K, MX_Only:MXOnly-1U-NoLED, symbol Switch:SW_Push
- added K54: L, MX_Only:MXOnly-1U-NoLED, symbol Switch:SW_Push
- added K55: Scln, MX_Only:MXOnly-1U-NoLED, symbol Switch:SW_Push
- added K56: Quote, MX_Only:MXOnly-1U-NoLED, symbol Switch:SW_Push
- added K57: Enter, MX_Only:MXOnly-2.25U-NoLED, symbol Switch:SW_Push
- added K58: End, MX_Only:MXOnly-1U-NoLED, symbol Switch:SW_Push
- added K59: Shift, MX_Only:MXOnly-1.25U-NoLED, symbol Switch:SW_Push
- added K6, K60: 1, MX_Only:MXOnly-1U-NoLED, symbol Switch:SW_Push
- added K61, K7: 2, MX_Only:MXOnly-1U-NoLED, symbol Switch:SW_Push
- added K62, K8: 3, MX_Only:MXOnly-1U-NoLED, symbol Switch:SW_Push
- added K63: Enter, MX_Only:MXOnly-2U-NoLED, symbol Switch:SW_Push
- added K64: Shift, MX_Only:MXOnly-2.25U-NoLED, symbol Switch:SW_Push
- added K65: Shift, MX_Only:MXOnly-1U-NoLED, symbol Switch:SW_Push
- added K66: Z, MX_Only:MXOnly-1U-NoLED, symbol Switch:SW_Push
- added K67: X, MX_Only:MXOnly-1U-NoLED, symbol Switch:SW_Push
- added K68: C, MX_Only:MXOnly-1U-NoLED, symbol Switch:SW_Push
- added K69: V, MX_Only:MXOnly-1U-NoLED, symbol Switch:SW_Push
- added K70: B, MX_Only:MXOnly-1U-NoLED, symbol Switch:SW_Push
- added K71: N, MX_Only:MXOnly-1U-NoLED, symbol Switch:SW_Push
- added K72: M, MX_Only:MXOnly-1U-NoLED, symbol Switch:SW_Push
- added K73: Comm, MX_Only:MXOnly-1U-NoLED, symbol Switch:SW_Push
- added K74, K82: Dot, MX_Only:MXOnly-1U-NoLED, symbol Switch:SW_Push
- added K76: Shift, MX_Only:MXOnly-1.75U-NoLED, symbol Switch:SW_Push
- added K77: Up, MX_Only:MXOnly-1U-NoLED, symbol Switch:SW_Push
- added K78: Home, MX_Only:MXOnly-1U-NoLED, symbol Switch:SW_Push
- added K79: Ctrl, MX_Only:MXOnly-1.5U-NoLED, symbol Switch:SW_Push
- added K80: Alt, MX_Only:MXOnly-1.5U-NoLED, symbol Switch:SW_Push
- added K81: 0, MX_Only:MXOnly-2U-NoLED, symbol Switch:SW_Push
- added K83: Ctrl, MX_Only:MXOnly-1.25U-NoLED, symbol Switch:SW_Push
- added K84: Win, MX_Only:MXOnly-1.25U-NoLED, symbol Switch:SW_Push
- added K85: Alt, MX_Only:MXOnly-1.25U-NoLED, symbol Switch:SW_Push
- added K86: Space, MX_Only:MXOnly-6.25U-NoLED, symbol Switch:SW_Push
- added K87: Alt, MX_Only:MXOnly-1U-NoLED, symbol Switch:SW_Push
- added K88: Win, MX_Only:MXOnly-1U-NoLED, symbol Switch:SW_Push
- added K89: Ctrl, MX_Only:MXOnly-1U-NoLED, symbol Switch:SW_Push
- added K90: Left, MX_Only:MXOnly-1U-NoLED, symbol Switch:SW_Push
- added K91: Down, MX_Only:MXOnly-1U-NoLED, symbol Switch:SW_Push
- added K92: Right, MX_Only:MXOnly-1U-NoLED, symbol Switch:SW_Push
- added R5: 22Ω, Custom_Footprints:R_0603_Annotated, symbol Device:R_Small
- added R6: 1MΩ, Custom_Footprints:R_0603_Annotated, symbol Device:R_Small
- added R7: 10kΩ, Custom_Footprints:R_0603_Annotated, symbol Device:R_Small
- C1: value 100nF -> 1μF; footprint (none) -> Custom_Footprints:C_0603_Annotated
- C2: value 100nF -> 10μF; footprint (none) -> Custom_Footprints:C_0603_Annotated
- C3: footprint (none) -> Custom_Footprints:C_0603_Annotated
- C4: value 10μF -> 100nF; footprint (none) -> Custom_Footprints:C_0603_Annotated
- C5: value 1μF -> 100nF; footprint (none) -> Custom_Footprints:C_0603_Annotated
- D1, D10, D11, D12, D13, D14, D15, D16, D17, D18, D19, D2, D20, D21, D22, D23, D24, D25, D26, D27, D28, D29, D3, D30, D31, D32, D33, D34, D35, D36, D37, D38, D39, D4, D40, D41, D42, D43, D44, D45, D46, D47, D48, D5, D6, D7, D8, D9: value BAV70 -> CCD; footprint Package_TO_SOT_SMD:SOT-23 -> Custom_Footprints:SOT-23_Annotated
- R1: value 22Ω -> 10kΩ; footprint (none) -> Custom_Footprints:R_0603_Annotated
- R2: value 22Ω -> 5.1kΩ; footprint (none) -> Custom_Footprints:R_0603_Annotated
- R3: value 10kΩ -> 5.1kΩ; footprint (none) -> Custom_Footprints:R_0603_Annotated
- R4: value 10kΩ -> 22Ω; footprint (none) -> Custom_Footprints:R_0603_Annotated
- RST1: footprint (none) -> Custom_Footprints:Tactile_Switch
- U1: value ATmega32U4-AU -> ATmega32U4; footprint Package_QFP:TQFP-44_10x10mm_P0.8mm -> Custom_Footprints:ATMEGA32U4_Annotated
- Y1: footprint (none) -> Custom_Footprints:Resonator_3Pin_Annotated
Connections:
- net +5V: now also C5.1, R1.1, F1.1; no longer C1.1, R3.1
- net DA+: now also R4.2; no longer R1.2
- net DA-: now also R5.2; no longer R2.2
- net DB+: now also R4.1, J1.A6 (D+), J1.B6 (D+); no longer R1.1
- net DB-: now also J1.A7 (D-), J1.B7 (D-), R5.1; no longer R2.1
- net GND: now also R2.1, R3.1, C6.1, J1.A1 (GND), J1.A12 (GND), J1.B1 (GND), J1.B12 (GND), R6.2, R7.1; no longer R4.1
- net col0: now also D11.3 (K), D21.3 (K), D31.3 (K), D41.3 (K); no longer D2.3 (K), D3.3 (K), D4.3 (K), D5.3 (K)
- net col1: now also D12.3 (K), D2.3 (K), D22.3 (K), D32.3 (K), D42.3 (K); no longer D10.3 (K), D6.3 (K), D7.3 (K), D8.3 (K), D9.3 (K)
- net col2: now also D23.3 (K), D3.3 (K), D33.3 (K), D43.3 (K); no longer D11.3 (K), D12.3 (K), D14.3 (K), D15.3 (K)
- net col3: now also D14.3 (K), D24.3 (K), D34.3 (K), D4.3 (K), D44.3 (K); no longer D16.3 (K), D17.3 (K), D18.3 (K), D19.3 (K), D20.3 (K)
- net col4: now also D15.3 (K), D25.3 (K), D35.3 (K), D5.3 (K); no longer D21.3 (K), D22.3 (K), D23.3 (K), D24.3 (K)
- net col5: now also D16.3 (K), D36.3 (K), D45.3 (K), D6.3 (K); no longer D25.3 (K), D27.3 (K), D28.3 (K), D29.3 (K)
- net col6: now also D17.3 (K), D27.3 (K), D37.3 (K), D7.3 (K); no longer D30.3 (K), D31.3 (K), D32.3 (K), D33.3 (K)
- net col7: now also D18.3 (K), D28.3 (K), D46.3 (K), D8.3 (K); no longer D34.3 (K), D35.3 (K), D36.3 (K), D37.3 (K)
- net col8: now also D19.3 (K), D29.3 (K), D47.3 (K), D9.3 (K); no longer D40.3 (K), D41.3 (K), D42.3 (K), D43.3 (K)
- net col9: now also D10.3 (K), D20.3 (K), D30.3 (K), D40.3 (K); no longer D44.3 (K), D45.3 (K), D46.3 (K), D47.3 (K)
- net row0: now also K1.1, K11.1, K13.1, K15.1, K17.1, K19.1, K3.1, K5.1, K7.1, K9.1
- net row1: now also K10.1, K12.1, K14.1, K16.1, K18.1, K2.1, K20.1, K21.1, K4.1, K6.1, K8.1
- net row2: now also K22.1, K24.1, K26.1, K28.1, K30.1, K32.1, K34.1, K36.1, K38.1
- net row3: now also K23.1, K25.1, K27.1, K29.1, K31.1, K33.1, K35.1, K37.1, K39.1, K40.1
- net row4: now also K41.1, K42.1, K44.1, K45.1, K47.1, K49.1, K51.1, K53.1, K55.1
- net row5: now also K43.1, K46.1, K48.1, K50.1, K52.1, K54.1, K56.1, K57.1, K58.1
- net row6: now also K59.1, K60.1, K62.1, K64.1, K66.1, K68.1, K70.1, K72.1, K74.1, K76.1, K77.1
- net row7: now also K61.1, K63.1, K65.1, K67.1, K69.1, K71.1, K73.1, K75.1, K78.1
- net row8: now also K81.1, K82.1, K83.1, K85.1, K86.1
- net row9: now also K84.1, K88.1, K90.1, K92.1
- net at D1.1 (A): now also K1.2
- net at D1.2 (A): now also K2.2
- net at D2.1 (A): now also K3.2
- net at D2.2 (A): now also K4.2
- net at D3.1 (A): now also K5.2
- net at D3.2 (A): now also K6.2
- net at D4.1 (A): now also K7.2
- net at D4.2 (A): now also K8.2
- net at D5.1 (A): now also K9.2
- net at D5.2 (A): now also K10.2
- net at D6.1 (A): now also K11.2
- net at D6.2 (A): now also K12.2
- net at D7.1 (A): now also K13.2
- net at D7.2 (A): now also K14.2
- net at D8.1 (A): now also K15.2
- net at D8.2 (A): now also K16.2
- net at D9.1 (A): now also K17.2
- net at D9.2 (A): now also K18.2, K21.2
- net at D10.1 (A): now also K19.2
- net at D10.2 (A): now also K20.2
- net at D11.1 (A): now also K22.2
- net at D11.2 (A): now also K23.2
- net at D12.1 (A): now also K24.2
- net at D12.2 (A): now also K25.2
- net at D13.1 (A): now also K26.2
- net at D13.2 (A): now also K27.2
- net at D14.1 (A): now also K28.2
- net at D14.2 (A): now also K29.2
- net at D15.1 (A): now also K30.2
- net at D15.2 (A): now also K31.2
- net at D16.1 (A): now also K32.2
- net at D16.2 (A): now also K33.2
- net at D17.1 (A): now also K34.2
- net at D17.2 (A): now also K35.2
- net at D18.1 (A): now also K36.2
- net at D18.2 (A): now also K37.2
- net at D19.1 (A): now also K38.2
- net at D19.2 (A): now also K39.2
- net at D20.2 (A): now also K40.2
- net at D21.1 (A): now also K42.2
- net at D21.2 (A): now also K43.2
- net at D22.1 (A): now also K44.2
- net at D23.1 (A): now also K41.2, K45.2
- net at D23.2 (A): now also K46.2
- net at D24.1 (A): now also K47.2
- net at D24.2 (A): now also K48.2
- net at D25.1 (A): now also K49.2
- net at D25.2 (A): now also K50.2
- net at D26.1 (A): now also K51.2
- net at D26.2 (A): now also K52.2
- net at D27.1 (A): now also K53.2
- net at D27.2 (A): now also K54.2
- net at D28.1 (A): now also K55.2
- net at D28.2 (A): now also K56.2
- net at D29.2 (A): now also K57.2
- net at D30.2 (A): now also K58.2
- net at D31.1 (A): now also K60.2
- net at D31.2 (A): now also K61.2
- net at D32.1 (A): now also K62.2
- net at D32.2 (A): now also K63.2
- net at D33.1 (A): now also K59.2, K64.2
- net at D33.2 (A): now also K65.2
- net at D34.1 (A): now also K66.2
- net at D34.2 (A): now also K67.2
- net at D35.1 (A): now also K68.2
- net at D35.2 (A): now also K69.2
- net at D36.1 (A): now also K70.2
- net at D36.2 (A): now also K71.2
- net at D37.1 (A): now also K72.2
- net at D37.2 (A): now also K73.2
- net at D38.1 (A): now also K74.2
- net at D38.2 (A): now also K75.2
- net at D39.1 (A): now also K76.2
- net at D40.1 (A): now also K77.2
- net at D40.2 (A): now also K78.2
- net at D41.1 (A): now also K81.2
- net at D42.1 (A): now also K82.2
- net at D43.1 (A): now also K83.2
- net at D43.2 (A): now also K84.2
- net at D44.1 (A): now also K85.2
- net at D45.1 (A): now also K86.2
- net at D46.2 (A): now also K88.2
- net at D46.1 (A): now also K80.2, K87.2
- net at D47.1 (A): now also K79.2, K89.2
- net at D47.2 (A): now also K90.2
- net at D48.1 (A): now also K91.2
- net at D48.2 (A): now also K92.2
- net at RST1.2, U1.13 (~RESET): now also R1.2; no longer R3.2
- net at U1.33 (~HWB~/PE2): now also R7.2; no longer R4.2
- net at U1.6 (UCAP): now also C1.1; no longer C5.1
- new net: K79.1, K80.1, K87.1, K89.1, K91.1
- new net: J1.A5 (CC1), R2.2
- new net: J1.B5 (CC2), R3.2
- new net: C6.2, J1.S1 (SHIELD), R6.1
- new net VCC: F1.2, J1.A4 (VBUS), J1.A9 (VBUS), J1.B4 (VBUS), J1.B9 (VBUS)
- no-connect marks 1 -> 3

Commit message: Route
Parts:
- removed J1: USB C, Custom_Footprints:Mid_Mount-USB_C_HandSoldering, symbol Connector:USB_C_Receptacle_USB2.0
- added J1: USB C, Custom_Footprints:Mid_Mount-USB_C_HandSoldering, symbol usb-type-c:USB2_C_Receptacle
- added J2: ISP, Custom_Footprints:ISP_Header_Annotated, symbol Connector:AVR-ISP-6
Connections:
- net +5V: now also J2.2 (VCC)
- net DB+: now also J1.A6 (D+), J1.B6 (D+)
- net DB-: now also J1.A7 (D-), J1.B7 (D-)
- net GND: now also J1.A1B12 (GND), J1.B1A12 (GND), J2.6 (GND)
- net VCC: now also J1.A4B9 (VBUS), J1.B4A9 (VBUS)
- net row0: now also K1.2, K11.2, K13.2, K15.2, K17.2, K19.2, K3.2, K5.2, K7.2, K9.2; no longer K1.1, K11.1, K13.1, K15.1, K17.1, K19.1, K3.1, K5.1, K7.1, K9.1
- net row1: now also K10.2, K12.2, K14.2, K16.2, K18.2, K2.2, K20.2, K21.2, K4.2, K6.2, K8.2; no longer K10.1, K12.1, K14.1, K16.1, K18.1, K2.1, K20.1, K21.1, K4.1, K6.1, K8.1
- net row2: now also K22.2, K24.2, K26.2, K28.2, K30.2, K32.2, K34.2, K36.2, K38.2; no longer K22.1, K24.1, K26.1, K28.1, K30.1, K32.1, K34.1, K36.1, K38.1
- net row3: now also K23.2, K25.2, K27.2, K29.2, K31.2, K33.2, K35.2, K37.2, K39.2, K40.2; no longer K23.1, K25.1, K27.1, K29.1, K31.1, K33.1, K35.1, K37.1, K39.1, K40.1
- net row4: now also K41.2, K42.2, K44.2, K45.2, K47.2, K49.2, K51.2, K53.2, K55.2; no longer K41.1, K42.1, K44.1, K45.1, K47.1, K49.1, K51.1, K53.1, K55.1
- net row5: now also K43.2, K46.2, K48.2, K50.2, K52.2, K54.2, K56.2, K57.2, K58.2; no longer K43.1, K46.1, K48.1, K50.1, K52.1, K54.1, K56.1, K57.1, K58.1
- net row6: now also K59.2, K60.2, K62.2, K64.2, K66.2, K68.2, K70.2, K72.2, K74.2, K76.2, K77.2; no longer K59.1, K60.1, K62.1, K64.1, K66.1, K68.1, K70.1, K72.1, K74.1, K76.1, K77.1
- net row7: now also K61.2, K63.2, K65.2, K67.2, K69.2, K71.2, K73.2, K75.2, K78.2; no longer K61.1, K63.1, K65.1, K67.1, K69.1, K71.1, K73.1, K75.1, K78.1
- net row8: now also K81.2, K82.2, K83.2, K85.2, K86.2; no longer K81.1, K82.1, K83.1, K85.1, K86.1
- net row9: now also K84.2, K88.2, K90.2, K92.2; no longer K84.1, K88.1, K90.1, K92.1
- net at D1.1 (A): now also K1.1; no longer K1.2
- net at D1.2 (A): now also K2.1; no longer K2.2
- net at D11.1 (A): now also K22.1; no longer K22.2
- net at D11.2 (A): now also K23.1; no longer K23.2
- net at D21.1 (A): now also K42.1; no longer K42.2
- net at D21.2 (A): now also K43.1; no longer K43.2
- net at D31.1 (A): now also K60.1; no longer K60.2
- net at D31.2 (A): now also K61.1; no longer K61.2
- net at D41.1 (A): no longer K81.2
- net at D41.2 (A): now also K81.1
- net at D2.1 (A): now also K3.1; no longer K3.2
- net at D2.2 (A): now also K4.1; no longer K4.2
- net at D12.1 (A): now also K24.1; no longer K24.2
- net at D12.2 (A): now also K25.1; no longer K25.2
- net at D22.1 (A): now also K44.1; no longer K44.2
- net at D32.1 (A): now also K63.1; no longer K62.2
- net at D32.2 (A): now also K62.1; no longer K63.2
- net at D42.1 (A): no longer K82.2
- net at D42.2 (A): now also K82.1
- net at D3.1 (A): now also K5.1; no longer K5.2
- net at D3.2 (A): now also K6.1; no longer K6.2
- net at D13.1 (A): now also K26.1; no longer K26.2
- net at D13.2 (A): now also K27.1; no longer K27.2
- net at D23.2 (A): now also K46.1; no longer K46.2
- net at D33.2 (A): now also K59.1, K64.1; no longer K65.2
- net at D43.1 (A): now also K84.1; no longer K83.2
- net at D43.2 (A): now also K83.1; no longer K84.2
- net at D4.1 (A): now also K7.1; no longer K7.2
- net at D4.2 (A): now also K8.1; no longer K8.2
- net at D14.1 (A): now also K28.1; no longer K28.2
- net at D14.2 (A): now also K29.1; no longer K29.2
- net at D24.1 (A): now also K47.1; no longer K47.2
- net at D24.2 (A): now also K48.1; no longer K48.2
- net at D34.1 (A): now also K66.1; no longer K66.2
- net at D34.2 (A): now also K67.1; no longer K67.2
- net at D44.1 (A): no longer K85.2
- net at D44.2 (A): now also K85.1
- net at D35.2 (A): now also K69.1; no longer K69.2
- net at D35.1 (A): now also K68.1; no longer K68.2
- net at D25.2 (A): now also K50.1; no longer K50.2
- net at D25.1 (A): now also K49.1; no longer K49.2
- net at D15.2 (A): now also K31.1; no longer K31.2
- net at D15.1 (A): now also K30.1; no longer K30.2
- net at D5.2 (A): now also K10.1; no longer K10.2
- net at D5.1 (A): now also K9.1; no longer K9.2
- net at D6.1 (A): now also K11.1; no longer K11.2
- net at D6.2 (A): now also K12.1; no longer K12.2
- net at D16.1 (A): now also K32.1; no longer K32.2
- net at D16.2 (A): now also K33.1; no longer K33.2
- net at D26.1 (A): now also K51.1; no longer K51.2
- net at D26.2 (A): now also K52.1; no longer K52.2
- net at D36.1 (A): now also K70.1; no longer K70.2
- net at D36.2 (A): now also K71.1; no longer K71.2
- net at D45.1 (A): no longer K86.2
- net at D45.2 (A): now also K86.1
- net at D37.2 (A): now also K73.1; no longer K73.2
- net at D37.1 (A): now also K72.1; no longer K72.2
- net at D27.2 (A): now also K54.1; no longer K54.2
- net at D27.1 (A): now also K53.1; no longer K53.2
- net at D17.2 (A): now also K35.1; no longer K35.2
- net at D17.1 (A): now also K34.1; no longer K34.2
- net at D7.2 (A): now also K14.1; no longer K14.2
- net at D7.1 (A): now also K13.1; no longer K13.2
- net at D8.1 (A): now also K15.1; no longer K15.2
- net at D8.2 (A): now also K16.1; no longer K16.2
- net at D18.1 (A): now also K36.1; no longer K36.2
- net at D18.2 (A): now also K37.1; no longer K37.2
- net at D28.1 (A): now also K55.1; no longer K55.2
- net at D28.2 (A): now also K56.1; no longer K56.2
- net at D38.1 (A): now also K74.1; no longer K74.2
- net at D38.2 (A): now also K75.1; no longer K75.2
- net at K80.2, K87.2: now also K79.2, K89.2, K91.2; no longer D46.1 (A)
- net at D46.2 (A): now also K80.1, K87.1; no longer K88.2
- net at D47.2 (A): now also K79.1, K89.1; no longer K90.2
- net at D39.1 (A): now also K76.1; no longer K76.2
- net at D29.2 (A): now also K57.1; no longer K57.2
- net at D19.2 (A): now also K39.1; no longer K39.2
- net at D19.1 (A): now also K38.1; no longer K38.2
- net at D9.1 (A): now also K17.1; no longer K17.2
- net at D10.1 (A): now also K19.1; no longer K19.2
- net at D10.2 (A): now also K20.1; no longer K20.2
- net at D20.2 (A): now also K40.1; no longer K40.2
- net at D30.2 (A): now also K58.1; no longer K58.2
- net at D40.1 (A): now also K77.1; no longer K77.2
- net at D40.2 (A): now also K78.1; no longer K78.2
- net at D48.1 (A): now also K92.1; no longer K91.2
- net at D48.2 (A): now also K91.1; no longer K92.2
- net MOSI: now reaches U1.10 (PB2)
- net MOSI: now also J2.4 (MOSI)
- net MISO: now reaches U1.11 (PB3)
- net MISO: now also J2.1 (MISO)
- net RST: now reaches R1.2, RST1.2, U1.13 (~RESET)
- net RST: now also J2.5 (~RST)
- net SCK: now reaches U1.9 (PB1)
- net SCK: now also J2.3 (SCK)
- net at R2.2: now also J1.A5 (CC1)
- net at R3.2: now also J1.B5 (CC2)
- net at C6.2, R6.1: now also J1.S1 (Shield)
- new net: D23.1 (A), K41.1, K45.1
- new net: D33.1 (A), K65.1
- new net: D46.1 (A), K88.1
- new net: D47.1 (A), K90.1
- new net: D9.2 (A), K18.1, K21.1
- no-connect marks 3 -> 1
Other:
- moved on the sheet: C6, F1, R2, R3, R6

Commit message: Finish Routing
Parts:
- added ENC1: ENC, Custom_Footprints:Rotary_Encoder, symbol Device:Rotary_Encoder_Switch
Connections:
- net row1 is gone; now on net S1: K10.2, K12.2, K14.2, K16.2, K18.2, K2.2, K20.2, K21.2, K4.2, K6.2, K8.2
- net GND: now also ENC1.C
- net col0: now also U1.30 (PB6)
- net col1: now also U1.31 (PC6)
- net col2: now also U1.32 (PC7)
- net col3: now also U1.36 (PF7)
- net col4: now also U1.37 (PF6)
- net col5: now also U1.38 (PF5)
- net col6: now also U1.39 (PF4)
- net col7: now also U1.40 (PF1)
- net col8: now also U1.41 (PF0)
- net col9: now also U1.18 (PD0)
- net row0: now also U1.19 (PD1)
- net row2: now also U1.29 (PB5)
- net row3: now also U1.12 (PB7)
- net row4: now also U1.21 (PD3)
- net row5: now also U1.22 (PD5)
- net row6: now also U1.26 (PD6)
- net row7: now also U1.25 (PD4)
- net row8: now also K79.2, K80.2, K87.2, K89.2, K91.2, U1.27 (PD7)
- net row9: now also U1.28 (PB4)
- net S2: now reaches D10.2 (A), K20.1
- net S2: now also ENC1.S2
- net ENCA: now reaches U1.1 (PE6)
- net ENCA: now also ENC1.A
- net S1: now reaches U1.20 (PD2)
- net S1: now also ENC1.S1
- net ENCB: now reaches U1.8 (PB0)
- net ENCB: now also ENC1.B
Changed lines of the file:
@@
 Comment4 ""
 $EndDescr
-Text GLabel 5450 6600 2    50   Input ~ 0
+Text GLabel 3900 6800 2    50   Input ~ 0
 row0
-Text GLabel 5450 6700 2    50   Input ~ 0
+Text GLabel 3900 6900 2    50   Input ~ 0
 row1
-Text GLabel 5450 6800 2    50   Input ~ 0
+Text GLabel 3900 6000 2    50   Input ~ 0
 row2
-Text GLabel 5450 6900 2    50   Input ~ 0
+Text GLabel 3900 6200 2    50   Input ~ 0
 row3
-Text GLabel 5450 7000 2    50   Input ~ 0
+Text GLabel 3900 7000 2    50   Input ~ 0
 row4
-Text GLabel 5450 7100 2    50   Input ~ 0
+Text GLabel 3900 7200 2    50   Input ~ 0
 row5
-Text GLabel 5450 7200 2    50   Input ~ 0
+Text GLabel 3900 7300 2    50   Input ~ 0
 row6
-Text GLabel 5450 7400 2    50   Input ~ 0
+Text GLabel 3900 7400 2    50   Input ~ 0
 row8
-Text GLabel 5450 7300 2    50   Input ~ 0
+Text GLabel 3900 7100 2    50   Input ~ 0
 row7
-Text GLabel 5450 7500 2    50   Input ~ 0
+Text GLabel 3900 5900 2    50   Input ~ 0
 row9
-Text GLabel 5800 6600 2    50   Input ~ 0
+Text GLabel 3900 6100 2    50   Input ~ 0
 col0
-Text GLabel 5800 6700 2    50   Input ~ 0
+Text GLabel 3900 6400 2    50   Input ~ 0
 col1
-Text GLabel 5800 6800 2    50   Input ~ 0
+Text GLabel 3900 6500 2    50   Input ~ 0
 col2
-Text GLabel 5800 6900 2    50   Input ~ 0
+Text GLabel 3900 8400 2    50   Input ~ 0
 col3
-Text GLabel 5800 7000 2    50   Input ~ 0
+Text GLabel 3900 8300 2    50   Input ~ 0
 col4
-Text GLabel 5800 7100 2    50   Input ~ 0
+Text GLabel 3900 8200 2    50   Input ~ 0
 col5
-Text GLabel 5800 7200 2    50   Input ~ 0
+Text GLabel 3900 8100 2    50   Input ~ 0
 col6
-Text GLabel 5800 7300 2    50   Input ~ 0
+Text GLabel 3900 8000 2    50   Input ~ 0
 col7
-Text GLabel 5800 7400 2    50   Input ~ 0
+Text GLabel 3900 7900 2    50   Input ~ 0
 col8
-Text GLabel 5800 7500 2    50   Input ~ 0
+Text GLabel 3900 6700 2    50   Input ~ 0
 col9
 $Comp
@@
 Text GLabel 11100 6450 2    50   Input ~ 0
 SCK
+$Comp
+L Device:Rotary_Encoder_Switch ENC1
+U 1 1 5F44433E
+P 20150 5200
+F 0 "ENC1" H 20150 5567 50  0000 C CNN
+F 1 "ENC" H 20150 5476 50  0000 C CNN
+F 2 "Custom_Footprints:Rotary_Encoder" H 20000 5360 50  0001 C CNN
+F 3 "~" H 20150 5460 50  0001 C CNN
+	1    20150 5200
+	1    0    0    -1
+$EndComp
+Text GLabel 20450 5100 2    50   Input ~ 0
+S1
+Text GLabel 20450 5300 2    50   Input ~ 0
+S2
+Text GLabel 19850 5100 0    50   Input ~ 0
+ENCA
+Text GLabel 19850 5300 0    50   Input ~ 0
+ENCB
+$Comp
+L power:GND #PWR018
+U 1 1 5F44B92D
+P 19450 5200
+F 0 "#PWR018" H 19450 4950 50  0001 C CNN
+F 1 "GND" H 19455 5027 50  0000 C CNN
+F 2 "" H 19450 5200 50  0001 C CNN
+F 3 "" H 19450 5200 50  0001 C CNN
+	1    19450 5200
+	1    0    0    -1
+$EndComp
+Wire Wire Line
+	19450 5200 19850 5200
+Text GLabel 20650 1400 2    50   Input ~ 0
+S1
+Text GLabel 20250 1400 1    50   Input ~ 0
+S2
+Text GLabel 3900 7700 2    50   Input ~ 0
+ENCA
+Text GLabel 3900 5500 2    50   Input ~ 0
+ENCB
+Wire Wire Line
+	11650 3500 15350 3500
+Connection ~ 11650 3500
 $EndSCHEMATC
