File: Southpaw/Southpaw.kicad_pcb (KiCad board)
At the start: 2 copper layers, 6.3 x 15.2 mm, 158 parts, among them J1 USB C, K1 Num, K10 5, K11 6, K12 7, K13 8, K14 9, K15 0, K16 Sub, K17 Plus, K18 Backspace, K19 Del, K2 Slash, K20 Mute, K21 Backspace, K22 7, K23 8, K24 9, K25 Plus, K26 Tab, K27 Q, K28 W, K29 E, K3 Mult, K30 R, K31 T, K32 Y, K33 U, K34 I, K35 O, K36 P, K37 LBrac, K38 Rbrac, K39 Pipe, K4 Sub, K40 Del, K41 SCaps, K42 4, K43 5, K44 6, K45 Caps, K46 A, K47 S, K48 D, K49 F, K5 Esc, K50 G, K51 H, K52 J, K53 K, K54 L, K55 Scln, K56 Quote, K57 Enter, K58 End, K59 Shift, K6 1, K60 1, K61 2, K62 3, K63 Enter, K64 Shift, K65 Shift, K66 Z, K67 X, K68 C, K69 V, K7 2, K70 B, K71 N, K72 M, K73 Comm, K74 Dot, K75 Slash, K76 Shift, K77 Up, K78 Home, K79 Ctrl, K8 3, K80 Alt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

Commit message: Route
Parts:
- added J2: ISP, Custom_Footprints:ISP_Header_Annotated, B.Cu at (394.2, 21.6)
- moved D40 336.4 mm to (388.1, 69.1), turned to 270 degrees
- moved U1 333.4 mm to (379.4, 40.5), turned to 270 degrees
- moved C5 331.9 mm to (384.2, 48.2)
- moved C4 330.0 mm to (389.2, 37.6)
- moved D48 321.2 mm to (388.1, 83.3), turned to 90 degrees
- moved D30 318.5 mm to (388.1, 49.2), turned to 270 degrees
- moved RST1 306.5 mm to (371.2, -3.00)
- moved D39 297.8 mm to (353.2, 68.3), turned to 270 degrees
- moved Y1 296.0 mm to (389.0, 40.4), turned to 90 degrees
- moved D20 289.8 mm to (388.1, 30.2), turned to 270 degrees
- moved D47 280.1 mm to (341.3, 79.4), turned to 90 degrees
- moved D10 277.9 mm to (388.1, 11.1), turned to 270 degrees
- moved R1 275.6 mm to (392.8, 37.6)
- moved D29 272.7 mm to (346.9, 49.2), turned to 270 degrees
- moved C2 266.5 mm to (381.0, 31.0), turned to 90 degrees
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Connections:
- net Net-(R1-Pad2) renamed RST
- J1 pad A1B12: (no net) -> GND
- J1 pad A4B9: (no net) -> VCC
- J1 pad B1A12: (no net) -> GND
- J1 pad B4A9: (no net) -> VCC
- K1 pad 1: row0 -> Net-(D1-Pad1)
- K1 pad 2: Net-(D1-Pad1) -> row0
- K10 pad 1: row1 -> Net-(D5-Pad2)
- K10 pad 2: Net-(D5-Pad2) -> row1
- K11 pad 1: row0 -> Net-(D6-Pad1)
- K11 pad 2: Net-(D6-Pad1) -> row0
- K12 pad 1: row1 -> Net-(D6-Pad2)
- K12 pad 2: Net-(D6-Pad2) -> row1
- K13 pad 1: row0 -> Net-(D7-Pad1)
- K13 pad 2: Net-(D7-Pad1) -> row0
- K14 pad 1: row1 -> Net-(D7-Pad2)
- K14 pad 2: Net-(D7-Pad2) -> row1
- K15 pad 1: row0 -> Net-(D8-Pad1)
- K15 pad 2: Net-(D8-Pad1) -> row0
- K16 pad 1: row1 -> Net-(D8-Pad2)
- K16 pad 2: Net-(D8-Pad2) -> row1
- K17 pad 1: row0 -> Net-(D9-Pad1)
- K17 pad 2: Net-(D9-Pad1) -> row0
- K18 pad 1: row1 -> Net-(D9-Pad2)
- K18 pad 2: Net-(D9-Pad2) -> row1
- K19 pad 1: row0 -> Net-(D10-Pad1)
- K19 pad 2: Net-(D10-Pad1) -> row0
- K2 pad 1: row1 -> Net-(D1-Pad2)
- K2 pad 2: Net-(D1-Pad2) -> row1
- K20 pad 1: row1 -> Net-(D10-Pad2)
- K20 pad 2: Net-(D10-Pad2) -> row1
- K21 pad 1: row1 -> Net-(D9-Pad2)
- K21 pad 2: Net-(D9-Pad2) -> row1
- K22 pad 1: row2 -> Net-(D11-Pad1)
- K22 pad 2: Net-(D11-Pad1) -> row2
- K23 pad 1: row3 -> Net-(D11-Pad2)
- K23 pad 2: Net-(D11-Pad2) -> row3
- K24 pad 1: row2 -> Net-(D12-Pad1)
- K24 pad 2: Net-(D12-Pad1) -> row2
- K25 pad 1: row3 -> Net-(D12-Pad2)
- K25 pad 2: Net-(D12-Pad2) -> row3
- K26 pad 1: row2 -> Net-(D13-Pad1)
- K26 pad 2: Net-(D13-Pad1) -> row2
- K27 pad 1: row3 -> Net-(D13-Pad2)
- K27 pad 2: Net-(D13-Pad2) -> row3
- K28 pad 1: row2 -> Net-(D14-Pad1)
- K28 pad 2: Net-(D14-Pad1) -> row2
- K29 pad 1: row3 -> Net-(D14-Pad2)
- K29 pad 2: Net-(D14-Pad2) -> row3
- K3 pad 1: row0 -> Net-(D2-Pad1)
- K3 pad 2: Net-(D2-Pad1) -> row0
- K30 pad 1: row2 -> Net-(D15-Pad1)
- K30 pad 2: Net-(D15-Pad1) -> row2
- K31 pad 1: row3 -> Net-(D15-Pad2)
- K31 pad 2: Net-(D15-Pad2) -> row3
- K32 pad 1: row2 -> Net-(D16-Pad1)
- K32 pad 2: Net-(D16-Pad1) -> row2
- K33 pad 1: row3 -> Net-(D16-Pad2)
- K33 pad 2: Net-(D16-Pad2) -> row3
- K34 pad 1: row2 -> Net-(D17-Pad1)
- K34 pad 2: Net-(D17-Pad1) -> row2
- K35 pad 1: row3 -> Net-(D17-Pad2)
- K35 pad 2: Net-(D17-Pad2) -> row3
- K36 pad 1: row2 -> Net-(D18-Pad1)
- K36 pad 2: Net-(D18-Pad1) -> row2
- K37 pad 1: row3 -> Net-(D18-Pad2)
- K37 pad 2: Net-(D18-Pad2) -> row3
- K38 pad 1: row2 -> Net-(D19-Pad1)
- K38 pad 2: Net-(D19-Pad1) -> row2
- K39 pad 1: row3 -> Net-(D19-Pad2)
- K39 pad 2: Net-(D19-Pad2) -> row3
- K4 pad 1: row1 -> Net-(D2-Pad2)
- K4 pad 2: Net-(D2-Pad2) -> row1
- K40 pad 1: row3 -> Net-(D20-Pad2)
- K40 pad 2: Net-(D20-Pad2) -> row3
- K41 pad 1: row4 -> Net-(D23-Pad1)
- K41 pad 2: Net-(D23-Pad1) -> row4
- K42 pad 1: row4 -> Net-(D21-Pad1)
- K42 pad 2: Net-(D21-Pad1) -> row4
- K43 pad 1: row5 -> Net-(D21-Pad2)
- K43 pad 2: Net-(D21-Pad2) -> row5
- K44 pad 1: row4 -> Net-(D22-Pad1)
- K44 pad 2: Net-(D22-Pad1) -> row4
- K45 pad 1: row4 -> Net-(D23-Pad1)
- K45 pad 2: Net-(D23-Pad1) -> row4
- K46 pad 1: row5 -> Net-(D23-Pad2)
- K46 pad 2: Net-(D23-Pad2) -> row5
- K47 pad 1: row4 -> Net-(D24-Pad1)
- K47 pad 2: Net-(D24-Pad1) -> row4
- K48 pad 1: row5 -> Net-(D24-Pad2)
- K48 pad 2: Net-(D24-Pad2) -> row5
- K49 pad 1: row4 -> Net-(D25-Pad1)
- K49 pad 2: Net-(D25-Pad1) -> row4
- K5 pad 1: row0 -> Net-(D3-Pad1)
- K5 pad 2: Net-(D3-Pad1) -> row0
- K50 pad 1: row5 -> Net-(D25-Pad2)
- K50 pad 2: Net-(D25-Pad2) -> row5
- K51 pad 1: row4 -> Net-(D26-Pad1)
- K51 pad 2: Net-(D26-Pad1) -> row4
- K52 pad 1: row5 -> Net-(D26-Pad2)
- K52 pad 2: Net-(D26-Pad2) -> row5
- K53 pad 1: row4 -> Net-(D27-Pad1)
- K53 pad 2: Net-(D27-Pad1) -> row4
- K54 pad 1: row5 -> Net-(D27-Pad2)
- K54 pad 2: Net-(D27-Pad2) -> row5
- K55 pad 1: row4 -> Net-(D28-Pad1)
- K55 pad 2: Net-(D28-Pad1) -> row4
- K56 pad 1: row5 -> Net-(D28-Pad2)
- K56 pad 2: Net-(D28-Pad2) -> row5
- K57 pad 1: row5 -> Net-(D29-Pad2)
- K57 pad 2: Net-(D29-Pad2) -> row5
- K58 pad 1: row5 -> Net-(D30-Pad2)
- K58 pad 2: Net-(D30-Pad2) -> row5
- K59 pad 1: row6 -> Net-(D33-Pad2)
- K59 pad 2: Net-(D33-Pad1) -> row6
- K6 pad 1: row1 -> Net-(D3-Pad2)
- K6 pad 2: Net-(D3-Pad2) -> row1
- K60 pad 1: row6 -> Net-(D31-Pad1)
- K60 pad 2: Net-(D31-Pad1) -> row6
- K61 pad 1: row7 -> Net-(D31-Pad2)
- K61 pad 2: Net-(D31-Pad2) -> row7
- K62 pad 1: row6 -> Net-(D32-Pad2)
- K62 pad 2: Net-(D32-Pad1) -> row6
- K63 pad 1: row7 -> Net-(D32-Pad1)
- K63 pad 2: Net-(D32-Pad2) -> row7
- K64 pad 1: row6 -> Net-(D33-Pad2)
- K64 pad 2: Net-(D33-Pad1) -> row6
- K65 pad 1: row7 -> Net-(D33-Pad1)
- K65 pad 2: Net-(D33-Pad2) -> row7
- K66 pad 1: row6 -> Net-(D34-Pad1)
- K66 pad 2: Net-(D34-Pad1) -> row6
- K67 pad 1: row7 -> Net-(D34-Pad2)
- K67 pad 2: Net-(D34-Pad2) -> row7
- K68 pad 1: row6 -> Net-(D35-Pad1)
- K68 pad 2: Net-(D35-Pad1) -> row6
- K69 pad 1: row7 -> Net-(D35-Pad2)
- K69 pad 2: Net-(D35-Pad2) -> row7
- K7 pad 1: row0 -> Net-(D4-Pad1)
- K7 pad 2: Net-(D4-Pad1) -> row0
- K70 pad 1: row6 -> Net-(D36-Pad1)
- K70 pad 2: Net-(D36-Pad1) -> row6
- K71 pad 1: row7 -> Net-(D36-Pad2)
- K71 pad 2: Net-(D36-Pad2) -> row7
- K72 pad 1: row6 -> Net-(D37-Pad1)
- K72 pad 2: Net-(D37-Pad1) -> row6
- K73 pad 1: row7 -> Net-(D37-Pad2)
- K73 pad 2: Net-(D37-Pad2) -> row7
- K74 pad 1: row6 -> Net-(D38-Pad1)
- K74 pad 2: Net-(D38-Pad1) -> row6
- K75 pad 1: row7 -> Net-(D38-Pad2)
- K75 pad 2: Net-(D38-Pad2) -> row7
- K76 pad 1: row6 -> Net-(D39-Pad1)
- K76 pad 2: Net-(D39-Pad1) -> row6
- K77 pad 1: row6 -> Net-(D40-Pad1)
- K77 pad 2: Net-(D40-Pad1) -> row6
- K78 pad 1: row7 -> Net-(D40-Pad2)
- K78 pad 2: Net-(D40-Pad2) -> row7
- K79 pad 1: Net-(K79-Pad1) -> Net-(D47-Pad2)
- K79 pad 2: Net-(D47-Pad1) -> Net-(K79-Pad2)
- K8 pad 1: row1 -> Net-(D4-Pad2)
- K8 pad 2: Net-(D4-Pad2) -> row1
- K80 pad 1: Net-(K79-Pad1) -> Net-(D46-Pad2)
- K80 pad 2: Net-(D46-Pad1) -> Net-(K79-Pad2)
- K81 pad 1: row8 -> Net-(D41-Pad2)
- K81 pad 2: Net-(D41-Pad1) -> row8
- K82 pad 1: row8 -> Net-(D42-Pad2)
- K82 pad 2: Net-(D42-Pad1) -> row8
- K83 pad 1: row8 -> Net-(D43-Pad2)
- K83 pad 2: Net-(D43-Pad1) -> row8
- K84 pad 1: row9 -> Net-(D43-Pad1)
- K84 pad 2: Net-(D43-Pad2) -> row9
- K85 pad 1: row8 -> Net-(D44-Pad2)
- K85 pad 2: Net-(D44-Pad1) -> row8
- K86 pad 1: row8 -> Net-(D45-Pad2)
- K86 pad 2: Net-(D45-Pad1) -> row8
- K87 pad 1: Net-(K79-Pad1) -> Net-(D46-Pad2)
- K87 pad 2: Net-(D46-Pad1) -> Net-(K79-Pad2)
- K88 pad 1: row9 -> Net-(D46-Pad1)
- K88 pad 2: Net-(D46-Pad2) -> row9
- K89 pad 1: Net-(K79-Pad1) -> Net-(D47-Pad2)
- K89 pad 2: Net-(D47-Pad1) -> Net-(K79-Pad2)
- K9 pad 1: row0 -> Net-(D5-Pad1)
- K9 pad 2: Net-(D5-Pad1) -> row0
- K90 pad 1: row9 -> Net-(D47-Pad1)
- K90 pad 2: Net-(D47-Pad2) -> row9
- K91 pad 1: Net-(K79-Pad1) -> Net-(D48-Pad2)
- K91 pad 2: Net-(D48-Pad1) -> Net-(K79-Pad2)
- K92 pad 1: row9 -> Net-(D48-Pad1)
- K92 pad 2: Net-(D48-Pad2) -> row9
- U1 pad 10: Net-(U1-Pad10) -> MOSI
- U1 pad 11: Net-(U1-Pad11) -> MISO
- U1 pad 9: Net-(U1-Pad9) -> SCK
Routing:
- net row7: track 0.00 -> 456.6 mm
- net row3: track 0.00 -> 451.5 mm
- net row1: track 0.00 -> 375.8 mm
- net row6: track 0.00 -> 365.7 mm
- net row0: track 0.00 -> 359.9 mm
- net row2: track 0.00 -> 328.4 mm
- net row5: track 0.00 -> 296.6 mm
- net row4: track 0.00 -> 295.2 mm
- net row9: track 0.00 -> 273.9 mm
- net row8: track 0.00 -> 149.6 mm
- net Net-(K79-Pad2): track 0.00 -> 85.9 mm
- net col8: track 0.00 -> 83.3 mm
- net col7: track 0.00 -> 78.1 mm
- net col3: track 0.00 -> 78.1 mm
- net col5: track 0.00 -> 76.8 mm
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- added copper zone on B.Cu, net GND
- added copper zone on F.Cu, net GND
Other:
- board size 6.3 x 15.2 mm -> 15.2 x 6.3 mm

Commit message: Finish Routing
Parts:
- added ENC1: ENC, Custom_Footprints:Rotary_Encoder, F.Cu at (395.9, 12.7)
- moved R4 252.4 mm to (382.4, 15.0), turned to 270 degrees
- moved R5 250.7 mm to (380.8, 15.0), turned to 270 degrees
- moved C6 227.6 mm to (373.9, 6.97)
- moved R6 227.6 mm to (375.5, 6.97)
- moved R3 224.1 mm to (384.2, 7.42)
- moved J1 224.1 mm to (381.4, -4.11)
- moved R2 223.9 mm to (379.2, 7.43)
- moved F1 215.8 mm to (384.0, 10.8), turned to 90 degrees
- moved RST1 62.4 mm to (382.0, 58.4), turned to 180 degrees
- moved J2 9.80 mm to (384.4, 21.4)
- moved R7 1.36 mm to (373.6, 48.1)
- moved C1 1.00 mm to (378.4, 31.0)
- moved C2 1.00 mm to (380.0, 31.0)
- moved C3 1.00 mm to (374.8, 31.0)
- moved C4 1.00 mm to (388.2, 37.6)
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Connections:
- net Net-(D10-Pad2) renamed S2
- K10 pad 2: row1 -> S1
- K12 pad 2: row1 -> S1
- K14 pad 2: row1 -> S1
- K16 pad 2: row1 -> S1
- K18 pad 2: row1 -> S1
- K2 pad 2: row1 -> S1
- K20 pad 2: row1 -> S1
- K21 pad 2: row1 -> S1
- K4 pad 2: row1 -> S1
- K6 pad 2: row1 -> S1
- K79 pad 2: Net-(K79-Pad2) -> row8
- K8 pad 2: row1 -> S1
- K80 pad 2: Net-(K79-Pad2) -> row8
- K87 pad 2: Net-(K79-Pad2) -> row8
- K89 pad 2: Net-(K79-Pad2) -> row8
- K91 pad 2: Net-(K79-Pad2) -> row8
- U1 pad 1: Net-(U1-Pad1) -> ENCA
- U1 pad 12: Net-(U1-Pad12) -> row3
- U1 pad 18: Net-(U1-Pad18) -> col9
- U1 pad 19: Net-(U1-Pad19) -> row0
- U1 pad 20: Net-(U1-Pad20) -> S1
- U1 pad 21: Net-(U1-Pad21) -> row4
- U1 pad 22: Net-(U1-Pad22) -> row5
- U1 pad 25: Net-(U1-Pad25) -> row7
- U1 pad 26: Net-(U1-Pad26) -> row6
- U1 pad 27: Net-(U1-Pad27) -> row8
- U1 pad 28: Net-(U1-Pad28) -> row9
- U1 pad 29: Net-(U1-Pad29) -> row2
- U1 pad 30: Net-(U1-Pad30) -> col0
- U1 pad 31: Net-(U1-Pad31) -> col1
- U1 pad 32: Net-(U1-Pad32) -> col2
- U1 pad 36: Net-(U1-Pad36) -> col3
- U1 pad 37: Net-(U1-Pad37) -> col4
- U1 pad 38: Net-(U1-Pad38) -> col5
- U1 pad 39: Net-(U1-Pad39) -> col6
- U1 pad 40: Net-(U1-Pad40) -> col7
- U1 pad 41: Net-(U1-Pad41) -> col8
- U1 pad 8: Net-(U1-Pad8) -> ENCB
Routing:
- net S1: track 0.00 -> 427.1 mm, vias 0 -> 1
- net row1: track 375.8 -> 0.00 mm
- net col0: track 69.2 -> 421.8 mm
- net col1: track 66.3 -> 381.8 mm, vias 0 -> 2
- net row8: track 149.6 -> 417.1 mm
- net col2: track 75.3 -> 337.8 mm, vias 0 -> 2
- net col3: track 78.1 -> 305.7 mm, vias 0 -> 2
- net col4: track 67.0 -> 256.3 mm, vias 0 -> 2
- net col5: track 76.8 -> 227.6 mm, vias 0 -> 2
- net row4: track 295.2 -> 412.0 mm, vias 0 -> 1
- net col6: track 67.0 -> 179.6 mm, vias 0 -> 2
- net +5V: track 16.7 -> 108.0 mm, vias 0 -> 6
- net Net-(K79-Pad2): track 85.9 -> 0.00 mm
- net row5: track 296.6 -> 377.5 mm, vias 0 -> 1
- net row0: track 359.9 -> 439.5 mm, vias 0 -> 1
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Other:
- board size 15.2 x 6.3 mm -> 395.3 x 106.5 mm

Commit message: Gerbers / Art
Parts:
- added G***: LOGO, Logo:RedPandaSitting_1050, B.Cu at (192.8, 86.5)
- added G***: LOGO, Logo:RedPandaArms1050, B.Cu at (254.2, 87.0)
- added REF**: 12x12MakerMark, Logo:12x12MakerMark, B.Cu at (397.2, 81.2)
Other:
- board text added: "Designed by : Swiftrax"
- board text added: "Made during the COVID-19 Pandemic"
- board text added: "Pandamic"
